File: Schematics/SerialClamp/SerialClamp.kicad_sch (KiCad schematic)
At the start: 11 parts, among them J4 USB_C_Receptacle_USB2.0, SW2 Power, U1 FT232RL, U3 LD1117S12TR_SOT223

Commit message: Added serial and started work on CH32
Parts:
- removed U1: FT232RL, symbol ames_new:FT232RL
- added C1, C2: 100nF, Capacitor_SMD:C_0805_2012Metric, symbol Device:C_Small
- added D1: LED_Small, LED_SMD:LED_0805_2012Metric, symbol Device:LED_Small
- added H1, H2: MountingHole, MountingHole:MountingHole_2.2mm_M2, symbol Mechanical:MountingHole
- added J2: Conn_01x05, Connector_PinHeader_2.54mm:PinHeader_1x05_P2.54mm_Vertical, symbol Connector_Generic:Conn_01x05
- added U1: CH340E, Package_SO:MSOP-10_3x3mm_P0.5mm, symbol Interface_USB:CH340E
- F1: footprint (none) -> Fuse:Fuse_0603_1608Metric
- RN1: value 1k -> 330
Connections:
- net D+: now also U1.1 (UD+)
- net D-: now also U1.2 (UD-)
- net RX: now also RN1.4 (R4.1), J2.3 (Pin_3), U1.9 (RXD)
- net TX: now also RN1.3 (R3.1), J2.2 (Pin_2), U1.8 (TXD)
- net VCC: now also RN1.1 (R1.1), J2.1 (Pin_1); no longer RN1.3 (R3.1), RN1.4 (R4.1)
- net VSS: now also C1.2, C2.2, D1.1 (K), J2.4 (Pin_4), U1.3 (GND)
- net VUSB: now also C1.1, U1.7 (VCC)
- net at D1.2 (A), RN1.5 (R4.2): no longer RN1.6 (R3.2)
- net LED: no longer names the net of RN1.2 (R2.1)
- net LED: no longer RN1.1 (R1.1)
- new net: D2.2 (A), RN1.6 (R3.2)
- new net: D1.2 (A), RN1.8 (R1.2)
- new net: C2.1, U1.10 (V3)
- new net Reset: J2.5 (Pin_5), U1.4 (~{RTS})
- now unconnected: RN1.7 (R2.2)
- no-connect marks 7 -> 11
Other:
- moved on the sheet: D1
