File: Schematics/CH32VClamp/CH32VClamp.kicad_pcb (KiCad board)
At the start: 2 copper layers, 54.9 x 14 mm, 29 parts, among them J1 USB_C_Receptacle_USB2.0, J2 PGM, J3 OPGM, Q1 SE4625-PandN, Q2 SE4625-PandN, SW2 SW_MEC_5E, U1 ESP32-S2, U2 AP1117-33, Y1 40MHz

Commit message: Decide on standard and started routing
Parts:
- removed J3: OPGM, Connector_PinHeader_2.54mm:PinHeader_2x05_P2.54mm_Horizontal
- added D1: LED_Small, LED_SMD:LED_0603_1608Metric, F.Cu at (207.8, 84.0)
- added J4: Prog, Connector_PinHeader_2.54mm:PinHeader_1x05_P2.54mm_Vertical, F.Cu at (219.2, 81.4)
Connections:
- Q1 pad 3: 3V3SW -> VCC003
- Q1 pad 8: 3V3SW -> VCC003
- Q2 pad 3: 5VSW -> VCC003
- Q2 pad 8: 5VSW -> VCC003
- RN4 pad 1: VBUS -> Net-(D1-A)
- RN4 pad 2: unconnected-(RN4-R2.1-Pad2) -> Net-(D1-A)
- RN4 pad 3: unconnected-(RN4-R3.1-Pad3) -> VBUS
- RN4 pad 6: unconnected-(RN4-R3.2-Pad6) -> Net-(Q2-G2)
- RN4 pad 7: unconnected-(RN4-R2.2-Pad7) -> ProgAct
- RN4 pad 8: Net-(Q2-G2) -> ProgAct
- U1 pad 8: unconnected-(U1-GPIO3-Pad8) -> ProgAct
Routing:
- net VDD: track 0.00 -> 35.7 mm
- net MULTI2: track 0.00 -> 32.2 mm, vias 0 -> 1
- net Net-(F1-Pad1): track 0.00 -> 31.7 mm, vias 0 -> 2
- net GPIO0: track 0.00 -> 15.2 mm
- net VCC003: track 0.00 -> 14.9 mm, vias 0 -> 1
- net VBUS: track 0.00 -> 13.9 mm
- net Net-(U1-XTAL_P): track 0.00 -> 12.7 mm, vias 0 -> 2
- net VCCCTL3: track 0.00 -> 12.0 mm, vias 0 -> 2
- net SWIO: track 0.00 -> 9.09 mm
- net SWCL: track 0.00 -> 8.11 mm
- net Net-(J1-CC2): track 0.00 -> 7.64 mm, vias 0 -> 2
- net VCCCTL5: track 0.00 -> 7.28 mm, vias 0 -> 2
- net Net-(U1-XTAL_N): track 0.00 -> 6.83 mm
- net Net-(J1-CC1): track 0.00 -> 6.77 mm
- net Net-(U1-LNA_IN): track 0.00 -> 5.46 mm, vias 0 -> 2
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
Commit message: Ordered CH32V Clamp V1
Parts:
- added kibuzzard-65DCFED4: G***, kibuzzard-65DCFED4, B.Cu at (215.3, 87.6)
- added kibuzzard-65DCFFD3: G***, kibuzzard-65DCFFD3, B.Cu at (195.9, 86.7)
- moved J4 10.2 mm to (219.2, 91.6), turned to 180 degrees
Connections:
- F1 pad 2: VUSB -> VBUS
- J1 pad A1: VSS -> GND
- J1 pad A12: VSS -> GND
- J1 pad B1: VSS -> GND
- J1 pad B12: VSS -> GND
- J1 pad S1: VSS -> GND
- RN1 pad 3: VSS -> GND
- RN1 pad 4: VSS -> GND
Routing:
- net GND: track 0.00 -> 88.5 mm, vias 0 -> 35
- net VDD: track 35.7 -> 84.0 mm, vias 0 -> 4
- net SWIO: track 9.09 -> 48.4 mm, vias 0 -> 1
- net SWCL: track 8.11 -> 47.3 mm, vias 0 -> 2
- net VCCCTL3: track 12.0 -> 46.2 mm, vias 2 -> 4
- net SWPUD: track 0.00 -> 29.9 mm, vias 0 -> 2
- net ProgAct: track 0.00 -> 29.7 mm, vias 0 -> 2
- net VCCCTL5: track 7.28 -> 36.8 mm, vias 2 -> 4
- net SWPUC: track 0.00 -> 25.6 mm, vias 0 -> 2
- net MULTI2: track 32.2 -> 43.2 mm
- net RX: track 0.00 -> 6.82 mm
- net TX: track 0.00 -> 5.65 mm
- net Net-(Q2-G2): track 2.37 -> 6.29 mm
- net Net-(U1-XTAL_P): track 12.7 -> 10.7 mm, vias 2 -> 0
- net VBUS: track 13.9 -> 15.9 mm
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- added copper zone on B.Cu, net GND
- added copper zone on F.Cu, net GND
